File: door_module/hardware/door_module.sch (KiCad schematic (older format))
At the start: 53 parts, among them J1 Raspberry Pi

Commit message: Small initial changes to Schematic
Signed-off-by: Juergen G. Schimmer <schimmi2@gmail.com>
Parts:
- removed J? (x2): Screw_Terminal_01x04, symbol Connector:Screw_Terminal_01x04
- removed U? (x4): LTV-817, Package_DIP:DIP-4_W7.62mm, symbol Isolator:LTV-817
- added J? (x3): Screw_Terminal_01x04, symbol Connector:Screw_Terminal_01x04
- added R? (x16): R, symbol Device:R
- added U? (x6): LTV-817, Package_DIP:DIP-4_W7.62mm, symbol Isolator:LTV-817
Connections:
- net labels added: RX_USB0, RX_USB1, RX_USB2, RX_USB3, TX_USB0, TX_USB1, TX_USB2, TX_USB3
- wire segments 118 -> 240
Other:
- moved on the sheet: C?, J1, J?, R?, U?

Commit message: Finalized Alpha Version of Door-Module Schematic
Signed-off-by: Juergen G. Schimmer <schimmi2@gmail.com>
Parts:
- removed J?: FT4232_2, symbol Connector:Conn_01x12_Male
- removed J?: FT4232_3, symbol Connector:Conn_01x12_Male
- removed J?: FT4232_4, symbol Connector:Conn_01x12_Male
- added C?: 10µ, symbol Device:CP
- added C?: 1µ, symbol Device:CP
- added C?: 100n, symbol Device:C
- added D? (x9): 1N4007, Diode_THT:D_DO-41_SOD81_P10.16mm_Horizontal, symbol Diode:1N4007
- added D? (x2): LED, symbol Device:LED
- added D?: ZPDxx, Diode_THT:D_DO-35_SOD27_P10.16mm_Horizontal, symbol Diode:ZPDxx
- added J? (x2): Screw_Terminal_01x02, symbol Connector:Screw_Terminal_01x02
- added J?: Conn_02x02_Odd_Even, symbol Connector_Generic:Conn_02x02_Odd_Even
- added J? (x3): FT4232_1, symbol Connector:Conn_01x12_Male
- added Q?: IRF7404, Package_SO:SOIC-8_3.9x4.9mm_P1.27mm, symbol Transistor_FET:IRF7404
- added Q?: IRF6614, Package_DirectFET:DirectFET_ST, symbol Transistor_FET:IRF6614
- added R? (x12): R, symbol Device:R
- added U? (x2): LTV-817, Package_DIP:DIP-4_W7.62mm, symbol Isolator:LTV-817
- added U?: LP2950-5.0_TO92, Package_TO_SOT_THT:TO-92_Inline, symbol Regulator_Linear:LP2950-5.0_TO92
Connections:
- net labels added: +12VA
- wire segments 240 -> 397
Other:
- moved on the sheet: C?, J?, R?, U?

Commit message: Change:	buffered serial outputs Change:	PoE added 25k Resistor Add:	Test points Add:	Annotations and Values Change:	Tidy up things a little
Signed-off-by: Juergen G. Schimmer <schimmi2@gmail.com>
Parts:
- removed J? (x2): Screw_Terminal_01x04, symbol Connector:Screw_Terminal_01x04
- removed R? (x8): R, symbol Device:R
- removed U? (x4): LTV-817, Package_DIP:DIP-4_W7.62mm, symbol Isolator:LTV-817
- added D13: 1N4007, Diode_THT:D_DO-41_SOD81_P10.16mm_Horizontal, symbol Diode:1N4007
- added D66, D67, D76, D77, D86, D87, D96, D97: 1N4148, Diode_THT:D_DO-35_SOD27_P7.62mm_Horizontal, symbol Diode:1N4148
- added J80, J?: Screw_Terminal_01x04, symbol Connector:Screw_Terminal_01x04
- added JP? (x8): SolderJumper_2_Bridged, symbol Jumper:SolderJumper_2_Bridged
- added Q66, Q76, Q86, Q96: BC557, Package_TO_SOT_THT:TO-92_Inline, symbol Transistor_BJT:BC557
- added R1: 25k, symbol Device:R
- added R67, R77, R87, R97: 470, symbol Device:R
- added R86, R96: 10k, symbol Device:R
- added R88, R91, R98, R?: 330, symbol Device:R
- added R92, R?: 3k3, symbol Device:R
- added TP61, TP62, TP63, TP64, TP65, TP66, TP67, TP68, TP69, TP71, TP72, TP73, TP74, TP75, TP76, TP77, TP78, TP79, TP81, TP82, TP83, TP84, TP85, TP86, TP87, TP88, TP89, TP91, TP92, TP93, TP94, TP95, TP96, TP97, TP98, TP99, TP_+48POE, TP_-48POE, TP_12VA, TP_3V3A, TP_5V, TP_5VA, TP_GND (x2), TP_GNDA: TestPoint, symbol Connector:TestPoint
- added U81, U82, U91, U?: LTV-817, Package_DIP:DIP-4_W7.62mm, symbol Isolator:LTV-817
- D10: renamed from D?; value ZPDxx -> ZPD24
- J61, J71, J81, J91: renamed from J?; symbol Connector:Conn_01x12_Male -> Connector:Conn_01x11_Male
- R11, R4, R66, R76: renamed from R?; value R -> 10k
- R12, R2: renamed from R?; value R -> 2k2
- R16, R36, R52, R53, R54, R61, R68, R71, R78: renamed from R?; value R -> 330
- R21, R46, R56, R57: renamed from R?; value R -> 470
- R26, R41, R51, R62, R72: renamed from R?; value R -> 3k3
- R3: renamed from R?; value R -> 2R2
- R31: renamed from R?; value R -> 33
- R58: renamed from R?; value R -> 390
- R59: renamed from R?; value R -> 220
- gave numbers to parts that had none: 58
Connections:
- net +12V: now also R1.2, TP_+48POE.1
- net +12VA: now also D13.2 (A), TP_12VA.1
- net +3.3VA: now also U61.4, U71.4, TP_3V3A.1, U81.4, U91.4
- net +3V3: no longer U62.4, U72.4
- net +5V: now also TP_5V.1
- net +5VA: now also J80.1 (Pin_1), J?.1 (Pin_1), TP_5VA.1; no longer U61.4, U71.4
- net GND: now also R92.1, R?.1, TP_GND.1, TP_GND.1, U81.2, U91.2
- net GNDA: now also R76.1, D67.2 (A), D77.2 (A), D87.2 (A), D97.2 (A), J80.2 (Pin_2), J?.2 (Pin_2), Q66.1 (C), Q76.1 (C), Q86.1 (C), Q96.1 (C), R67.1, R77.1, R86.2, R87.1, R96.1, R97.1, TP_GNDA.1, U82.2, U?.2; no longer R76.2
- net RX_USB0: now also R?.2, TP62.1, TP82.1, U82.3; no longer J71.4 (Pin_4), J81.4 (Pin_4), J91.4 (Pin_4)
- net RX_USB1: now also J71.4 (Pin_4), R92.2, TP72.1, TP92.1, U?.3
- net RX_USB2: now also J81.4 (Pin_4)
- net RX_USB3: now also J91.4 (Pin_4)
- net TX_USB0: now also R?.1, TP61.1, TP81.1; no longer J71.3 (Pin_3), J81.3 (Pin_3), J91.3 (Pin_3)
- net TX_USB1: now also J71.3 (Pin_3), R91.1, TP71.1, TP91.1
- net TX_USB2: now also J81.3 (Pin_3)
- net TX_USB3: now also J91.3 (Pin_3)
- net at R66.1, U61.3: now also D66.2 (A), Q66.2 (B), TP69.1; no longer J60.3 (Pin_3)
- net at R68.1, U62.1: now also D67.1 (K)
- net +5VP: now reaches J61.1 (Pin_1)
- net +5VP: now also J71.1 (Pin_1), J81.1 (Pin_1), J91.1 (Pin_1)
- net at J61.10 (Pin_10): now also TP67.1
- net at J61.11 (Pin_11): now also TP68.1
- net +3.3VP: now reaches J61.2 (Pin_2)
- net +3.3VP: now also J71.2 (Pin_2), J81.2 (Pin_2), J91.2 (Pin_2), U62.4, U72.4, U82.4, U?.4
- net at J61.6 (Pin_6): now also JP?.2 (B), TP63.1; no longer J61.7 (Pin_7)
- net at J61.8 (Pin_8): now also JP?.2 (B), TP65.1; no longer J61.9 (Pin_9)
- net at R78.1, U72.1: now also D77.1 (K)
- net at C11.1, D11.2 (A), D12.1 (K)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: now also D13.1 (K)
- net at D1.1 (K), D2.1 (K), D7.2 (A)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: now also R1.1, TP_-48POE.1
- net at J71.10 (Pin_10): now also TP77.1
- net at J71.11 (Pin_11): now also TP78.1
- net at J71.6 (Pin_6): now also JP?.2 (B), TP73.1; no longer J71.7 (Pin_7)
- net at J71.8 (Pin_8): now also JP?.2 (B), TP75.1; no longer J71.9 (Pin_9)
- net at J81.10 (Pin_10): now also TP87.1
- net at J81.11 (Pin_11): now also TP88.1
- net at J81.6 (Pin_6): now also JP?.2 (B), TP83.1; no longer J81.7 (Pin_7)
- net at J81.8 (Pin_8): now also JP?.2 (B), TP85.1; no longer J81.9 (Pin_9)
- net at J91.10 (Pin_10): now also TP97.1
- net at J91.11 (Pin_11): now also TP98.1
- net at J91.6 (Pin_6): now also JP?.2 (B), TP93.1; no longer J91.7 (Pin_7)
- net at J91.8 (Pin_8): now also JP?.2 (B), TP95.1; no longer J91.9 (Pin_9)
- new net: D66.1 (K), J60.3 (Pin_3), Q66.3 (E), R67.2
- new net: J61.7 (Pin_7), JP?.1 (A), TP64.1
- new net: J61.9 (Pin_9), JP?.1 (A), TP66.1
- new net: D76.2 (A), Q76.2 (B), R76.2, TP79.1, U71.3
- new net: D76.1 (K), J70.3 (Pin_3), Q76.3 (E), R77.2
- new net: J71.7 (Pin_7), JP?.1 (A), TP74.1
- new net: J71.9 (Pin_9), JP?.1 (A), TP76.1
- new net: J81.7 (Pin_7), JP?.1 (A), TP84.1
- new net: J81.9 (Pin_9), JP?.1 (A), TP86.1
- new net: J91.7 (Pin_7), JP?.1 (A), TP94.1
- new net: J91.9 (Pin_9), JP?.1 (A), TP96.1
- new net: D87.1 (K), R88.1, U82.1
- new net: R?.2, U81.1
- new net: D86.2 (A), Q86.2 (B), R86.1, TP89.1, U81.3
- new net: J80.4 (Pin_4), R88.2
- new net: D86.1 (K), J80.3 (Pin_3), Q86.3 (E), R87.2
- new net: D97.1 (K), R98.1, U?.1
- new net: R91.2, U91.1
- new net: D96.2 (A), Q96.2 (B), R96.2, TP99.1, U91.3
- new net: J?.4 (Pin_4), R98.2
- new net: D96.1 (K), J?.3 (Pin_3), Q96.3 (E), R97.2
Other:
- moved on the sheet: C1, C2, C21, C22, C23, C24, C3, C4, C5, C6, C7, C8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

Commit message: First Placement of door_module PCB Minor changes to schematic
Signed-off-by: Juergen G. Schimmer <schimmi2@gmail.com>
Parts:
- C1: footprint (none) -> Capacitor_THT:CP_Radial_D13.0mm_P7.50mm
- C11, C21, C22, C23, C24, C3: footprint (none) -> Capacitor_THT:CP_Radial_D14.0mm_P7.50mm
- C2, C4, C5, C7, C9: footprint (none) -> Capacitor_THT:C_Disc_D3.0mm_W2.0mm_P2.50mm
- C6: footprint (none) -> Capacitor_THT:CP_Radial_D5.0mm_P2.00mm
- C8: footprint (none) -> Capacitor_THT:CP_Radial_Tantal_D5.5mm_P2.50mm
- D11, D9: footprint (none) -> LED_THT:LED_D5.0mm
- J1: footprint (none) -> Connector_PinSocket_2.54mm:PinSocket_2x40_P2.54mm_Horizontal
- J10, J20, J30, J40: footprint (none) -> Connector_Phoenix_MSTB:PhoenixContact_MSTBA_2,5_2-G-5,08_1x02_P5.08mm_Horizontal
- J14, J15, J17, J18, J6, J7, J8, J9: footprint (none) -> Connector_Wire:SolderWirePad_1x02_P3.81mm_Drill0.8mm
- J2: footprint (none) -> Connector_PinHeader_2.54mm:PinHeader_2x02_P2.54mm_Vertical
- J3: renamed from J2; footprint (none) -> Connector_RJ:RJ45_Wuerth_7499010121A_Horizontal
- J50: footprint (none) -> Connector_Phoenix_MSTB:PhoenixContact_MSTBA_2,5_6-G-5,08_1x06_P5.08mm_Horizontal
- J60, J70, J80: footprint (none) -> Connector_Phoenix_MSTB:PhoenixContact_MSTBA_2,5_4-G-5,08_1x04_P5.08mm_Horizontal
- J61, J71, J81, J91: footprint (none) -> Connector_PinSocket_2.54mm:PinSocket_1x11_P2.54mm_Vertical
- J90: renamed from J?; footprint (none) -> Connector_Phoenix_MSTB:PhoenixContact_MSTBA_2,5_4-G-5,08_1x04_P5.08mm_Horizontal
- JP61, JP62, JP71, JP72, JP81, JP82, JP91, JP92: renamed from JP?; footprint (none) -> Jumper:SolderJumper-2_P1.3mm_Bridged_Pad1.0x1.5mm
- R1, R11, R12, R16, R2, R21, R26, R3, R31, R36, R4, R41, R46, R51, R52, R53, R54, R56, R57, R58, R59, R61, R62, R66, R67, R68, R71, R72, R76, R77, R78, R86, R87, R88, R91, R92, R96, R97, R98: footprint (none) -> Resistor_THT:R_Axial_DIN0207_L6.3mm_D2.5mm_P10.16mm_Horizontal
- R81, R82: renamed from R?; footprint (none) -> Resistor_THT:R_Axial_DIN0207_L6.3mm_D2.5mm_P10.16mm_Horizontal
- TP61, TP62, TP63, TP64, TP65, TP66, TP67, TP68, TP69, TP71, TP72, TP73, TP74, TP75, TP76, TP77, TP78, TP79, TP81, TP82, TP83, TP84, TP85, TP86, TP87, TP88, TP89, TP91, TP92, TP93, TP94, TP95, TP96, TP97, TP98, TP99: footprint (none) -> TestPoint:TestPoint_Loop_D2.60mm_Drill1.6mm_Beaded
- TP_+48POE1: renamed from TP_+48POE; footprint (none) -> TestPoint:TestPoint_Loop_D2.60mm_Drill1.6mm_Beaded
- TP_-48POE1: renamed from TP_-48POE; footprint (none) -> TestPoint:TestPoint_Loop_D2.60mm_Drill1.6mm_Beaded
- TP_12VA1: renamed from TP_12VA; footprint (none) -> TestPoint:TestPoint_Loop_D2.60mm_Drill1.6mm_Beaded
- TP_3V3A1: renamed from TP_3V3A; footprint (none) -> TestPoint:TestPoint_Loop_D2.60mm_Drill1.6mm_Beaded
- TP_5V1: renamed from TP_5V; footprint (none) -> TestPoint:TestPoint_Loop_D2.60mm_Drill1.6mm_Beaded
- TP_5VA1: renamed from TP_5VA; footprint (none) -> TestPoint:TestPoint_Loop_D2.60mm_Drill1.6mm_Beaded
- TP_GND1, TP_GND2: renamed from TP_GND; footprint (none) -> TestPoint:TestPoint_Loop_D2.60mm_Drill1.6mm_Beaded
- TP_GNDA1: renamed from TP_GNDA; footprint (none) -> TestPoint:TestPoint_Loop_D2.60mm_Drill1.6mm_Beaded
- U1: footprint Converter_DCDC:Converter_DCDC_muRata_NMAxxxxSC_THT -> Package_SIP:PowerIntegrations_eSIP-7F
- gave numbers to parts that had none: 1
Connections:
- net RX_USB0: no longer R82.2, TP82.1, U82.3
- net RX_USB1: no longer R92.2, TP92.1, U1001.3
- net RX_USB2: now also R82.2, TP82.1, U82.3
- net RX_USB3: now also R92.2, TP92.1, U1001.3
- net TX_USB0: no longer R81.1, TP81.1
- net TX_USB1: no longer R91.1, TP91.1
- net TX_USB2: now also R81.1, TP81.1
- net TX_USB3: now also R91.1, TP91.1
- no-connect marks 1 -> 21

Commit message: First alpha PCB
Signed-off-by: Juergen G. Schimmer <schimmi2@gmail.com>
Parts:
- removed D10: ZPD24, Diode_THT:D_DO-35_SOD27_P10.16mm_Horizontal, symbol Diode:ZPDxx
- removed D2, D3, D4, D5, D6, D7, D8: 1N4007, Diode_THT:D_DO-41_SOD81_P10.16mm_Horizontal, symbol Diode:1N4007
- removed D9: LED, LED_THT:LED_D5.0mm, symbol Device:LED
- removed Q2: IRF6614, Package_DirectFET:DirectFET_ST, symbol Transistor_FET:IRF6614
- removed R1: 25k, Resistor_THT:R_Axial_DIN0207_L6.3mm_D2.5mm_P10.16mm_Horizontal, symbol Device:R
- removed R2: 2k2, Resistor_THT:R_Axial_DIN0207_L6.3mm_D2.5mm_P10.16mm_Horizontal, symbol Device:R
- removed R3: 2R2, Resistor_THT:R_Axial_DIN0207_L6.3mm_D2.5mm_P10.16mm_Horizontal, symbol Device:R
- removed R4: 10k, Resistor_THT:R_Axial_DIN0207_L6.3mm_D2.5mm_P10.16mm_Horizontal, symbol Device:R
- removed TP_+48POE1, TP_-48POE1, TP_GND2: TestPoint, TestPoint:TestPoint_Loop_D2.60mm_Drill1.6mm_Beaded, symbol Connector:TestPoint
- added J21, J22, J23, J24, J26, J27, J28: Conn_01x01_Male, Connector_PinHeader_2.54mm:PinHeader_1x01_P2.54mm_Vertical, symbol Connector:Conn_01x01_Male
- added J41, J42: Screw_Terminal_01x02, Connector_Phoenix_MSTB:PhoenixContact_MSTBA_2,5_2-G-5,08_1x02_P5.08mm_Horizontal, symbol Connector:Screw_Terminal_01x02
- added R41, R42: 470, Resistor_THT:R_Axial_DIN0207_L6.3mm_D2.5mm_P10.16mm_Horizontal, symbol Device:R
- added R46, R47: 3k3, Resistor_THT:R_Axial_DIN0207_L6.3mm_D2.5mm_P10.16mm_Horizontal, symbol Device:R
- added U41, U42: LTV-817, Package_DIP:DIP-4_W7.62mm, symbol Isolator:LTV-817
- J1: footprint Connector_PinSocket_2.54mm:PinSocket_2x40_P2.54mm_Horizontal -> Connector_PinSocket_2.54mm:PinSocket_2x20_P2.54mm_Vertical
- J61, J71, J81, J91: footprint Connector_PinSocket_2.54mm:PinSocket_1x11_P2.54mm_Vertical -> Connector_PinSocket_2.54mm:PinSocket_1x12_P2.54mm_Vertical; symbol Connector:Conn_01x11_Male -> Connector:Conn_01x12_Male
- Q11: footprint Package_SO:SOIC-8_3.9x4.9mm_P1.27mm -> Package_TO_SOT_THT:TO-220-3_Vertical; symbol Transistor_FET:IRF7404 -> Transistor_FET:IRF9540N
- TP61, TP62, TP63, TP64, TP65, TP66, TP67, TP68, TP69, TP71, TP72, TP73, TP74, TP75, TP76, TP77, TP78, TP79, TP81, TP82, TP83, TP84, TP85, TP86, TP87, TP88, TP89, TP91, TP92, TP93, TP94, TP95, TP96, TP97, TP98, TP99: footprint TestPoint:TestPoint_Loop_D2.60mm_Drill1.6mm_Beaded -> TestPoint:TestPoint_Loop_D1.80mm_Drill1.0mm_Beaded
- U1: footprint Package_SIP:PowerIntegrations_eSIP-7F -> Package_SIP:SIP9_Housing_BigPads
- renumbered J30 to J31, J40 to J32, R46 to R32, R41 to R37, U41 to U32
Connections:
- net +12V: now also D1.1 (K), J26.1 (Pin_1); no longer J3.4 (Pin_4), J3.5 (Pin_5)
- net +3V3: now also U41.4, U42.4
- net +5VA: now also U41.1, U42.1
- net BELL_BUTTON: now also J1.11 (Pin_11); no longer J1.7 (Pin_7)
- net BELL_LED_B: now also J1.3 (Pin_3); no longer J1.15 (Pin_15)
- net BELL_LED_G: now also J1.5 (Pin_5); no longer J1.13 (Pin_13)
- net BELL_LED_R: now also J1.7 (Pin_7); no longer J1.11 (Pin_11)
- net DOOR_CLOSER: now also J1.33 (Pin_33); no longer J1.12 (Pin_12)
- net FB_MAGNET: now also J1.21 (Pin_21); no longer J1.18 (Pin_18)
- net FB_STRIKE: now also J1.23 (Pin_23); no longer J1.16 (Pin_16)
- net GND: now also J61.12 (Pin_12), J71.12 (Pin_12), J81.12 (Pin_12), J91.12 (Pin_12), J27.1 (Pin_1), R46.1, R47.1
- net GNDA: now also J41.2 (Pin_2), J42.2 (Pin_2)
- net STRIKE: now also J1.37 (Pin_37); no longer J1.22 (Pin_22)
- net at C11.1, D11.2 (A), D12.1 (K)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: no longer Q11.1 (S), Q11.2 (S)
- net at D11.1 (K), R11.2, R12.1: now also Q11.1 (G); no longer Q11.4 (G)
- net at J2.1 (Pin_1): now also J21.1 (Pin_1); no longer D1.2 (A)
- net at J2.2 (Pin_2): now also J23.1 (Pin_1)
- net at J2.3 (Pin_3): now also J22.1 (Pin_1)
- net at J2.4 (Pin_4): now also J24.1 (Pin_1)
- new net: D12.2 (A), J10.2 (Pin_2), Q11.2 (D)
- new net: R41.1, U41.2
- new net: R42.1, U42.2
- new net: J41.1 (Pin_1), R41.2
- new net: J42.1 (Pin_1), R42.2
- new net GPIO1: J1.12 (Pin_12)
- new net GPIO4: J1.16 (Pin_16)
- new net GPIO5: J1.18 (Pin_18)
- new net GPIO6: J1.22 (Pin_22)
- new net Sabotage1: J1.15 (Pin_15), R46.2, U41.3
- new net Sabotage2: J1.13 (Pin_13), R47.2, U42.3
- new net bl: D1.2 (A), J3.4 (Pin_4), J3.5 (Pin_5)
Other:
- moved on the sheet: C1, C11, C2, C21, C22, C23, C24, C3, C4, C5, C6, C7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
